File: hardware/hi_sense.kicad_sch (KiCad schematic)
At the start: 9 parts, among them U1 PC817

Commit message: add enable timer in logic block
Parts:
- C5: value C -> ??
- D5: value D_Zener -> ??
- R10, R3, R4, R5, R7, R9: value R_US -> ??
Changed lines of the file:
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@@
 			)
 		)
-		(property "Value" "R_US"
+		(property "Value" "??"
 			(at 68.58 34.29 90)
 			(show_name no)
@@
 			)
 		)
-		(property "Value" "R_US"
+		(property "Value" "??"
 			(at 58.42 34.29 90)
 			(show_name no)
@@
 			)
 		)
-		(property "Value" "D_Zener"
+		(property "Value" "??"
 			(at 107.95 46.9899 90)
 			(show_name no)
@@
 			)
 		)
-		(property "Value" "R_US"
+		(property "Value" "??"
 			(at 77.47 48.2599 0)
 			(show_name no)
@@
 			)
 		)
-		(property "Value" "C"
+		(property "Value" "??"
 			(at 95.25 48.2599 0)
 			(show_name no)
@@
 			)
 		)
-		(property "Value" "R_US"
+		(property "Value" "??"
 			(at 48.26 34.29 90)
 			(show_name no)
@@
 			)
 		)
-		(property "Value" "R_US"
+		(property "Value" "??"
 			(at 125.73 44.4499 0)
 			(show_name no)
@@
 			)
 		)
-		(property "Value" "R_US"
+		(property "Value" "??"
 			(at 149.86 44.4499 0)
 			(show_name no)
