File: hardware/lv_logic.kicad_sch (KiCad schematic)
At the start: 14 parts, among them IC2 CD4081BM96, IC3 CD40106BM96, IC5 CD4071BM96, Q4 NMOS

Commit message: start power supply and logic sizing
Parts:
- IC2, IC3, IC5: footprint SOIC127P600X175-14N -> Library_Loader:SOIC127P600X175-14N
- R18: value ?? -> 10k
Connections:
- net GND: now also IC2.12 (G), IC2.13 (H), IC5.12 (G), IC5.13 (H)
- no-connect marks 6 -> 7
Changed lines of the file:
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@@
 	)
 	(junction
+		(at 153.67 133.35)
+		(diameter 0)
+		(color 0 0 0 0)
+	)
+	(junction
 		(at 118.11 133.35)
 		(diameter 0)
@@
 	)
 	(junction
+		(at 157.48 91.44)
+		(diameter 0)
+		(color 0 0 0 0)
+	)
+	(junction
 		(at 165.1 59.69)
 		(diameter 0)
@@
 		(at 151.13 128.27)
 	)
+	(no_connect
+		(at 151.13 93.98)
+	)
 	(wire
 		(pts
@@
 	(wire
 		(pts
+			(xy 151.13 91.44) (xy 157.48 91.44)
+		)
+		(stroke
+			(width 0)
+			(type default)
+		)
+	)
+	(wire
+		(pts
 			(xy 118.11 133.35) (xy 118.11 135.89)
 		)
@@
 	(wire
 		(pts
+			(xy 151.13 88.9) (xy 157.48 88.9)
+		)
+		(stroke
+			(width 0)
+			(type default)
+		)
+	)
+	(wire
+		(pts
 			(xy 123.19 71.12) (xy 119.38 71.12)
 		)
@@
 	(wire
 		(pts
+			(xy 157.48 91.44) (xy 157.48 102.87)
+		)
+		(stroke
+			(width 0)
+			(type default)
+		)
+	)
+	(wire
+		(pts
+			(xy 157.48 88.9) (xy 157.48 91.44)
+		)
+		(stroke
+			(width 0)
+			(type default)
+		)
+	)
+	(wire
+		(pts
 			(xy 120.65 99.06) (xy 113.03 99.06)
 		)
@@
 	(wire
 		(pts
-			(xy 153.67 125.73) (xy 153.67 130.81)
+			(xy 153.67 125.73) (xy 153.67 133.35)
 		)
 		(stroke
@@
 			)
 		)
-		(property "Footprint" "SOIC127P600X175-14N"
+		(property "Footprint" "Library_Loader:SOIC127P600X175-14N"
 			(at 147.32 181.28 0)
 			(hide yes)
@@
 			)
 		)
-		(property "Footprint" "SOIC127P600X175-14N"
+		(property "Footprint" "Library_Loader:SOIC127P600X175-14N"
 			(at 147.32 215.57 0)
 			(hide yes)
@@
 	)
 	(symbol
+		(lib_id "power:GND")
+		(at 157.48 102.87 0)
+		(unit 1)
+		(body_style 1)
+		(exclude_from_sim no)
+		(in_bom yes)
+		(on_board yes)
+		(in_pos_files yes)
+		(dnp no)
+		(fields_autoplaced yes)
+		(property "Reference" "#PWR049"
+			(at 157.48 109.22 0)
+			(hide yes)
+			(show_name no)
+			(do_not_autoplace no)
+			(effects
+				(font
+					(size 1.27 1.27)
+				)
+			)
+		)
+		(property "Value" "GND"
+			(at 157.48 107.95 0)
+			(show_name no)
+			(do_not_autoplace no)
+			(effects
+				(font
+					(size 1.27 1.27)
+				)
+			)
+		)
+		(property "Footprint" ""
+			(at 157.48 102.87 0)
+			(hide yes)
+			(show_name no)
+			(do_not_autoplace no)
+			(effects
+				(font
+					(size 1.27 1.27)
+				)
+			)
+		)
+		(property "Datasheet" ""
+			(at 157.48 102.87 0)
+			(hide yes)
+			(show_name no)
+			(do_not_autoplace no)
+			(effects
+				(font
+					(size 1.27 1.27)
+				)
+			)
+		)
+		(property "Description" "Power symbol creates a global label with name \"GND\" , ground"
+			(at 157.48 102.87 0)
+			(hide yes)
+			(show_name no)
+			(do_not_autoplace no)
+			(effects
+				(font
+					(size 1.27 1.27)
+				)
+			)
+		)
+		(pin "1"
+		)
+		(instances
+			(project "precharge-controller"
+				(path "/d0dc5348-c362-4b06-85a5-76de80ed7055/56fb71d1-0eb8-422f-888e-b936ea8ae617"
+					(reference "#PWR049")
+					(unit 1)
+				)
+			)
+		)
+	)
+	(symbol
 		(lib_id "power:+12V")
 		(at 67.31 97.79 90)
@@
 			)
 		)
-		(property "Value" "??"
+		(property "Value" "10k"
 			(at 121.92 81.2799 0)
 			(show_name no)
@@
 			)
 		)
-		(property "Footprint" "SOIC127P600X175-14N"
+		(property "Footprint" "Library_Loader:SOIC127P600X175-14N"
 			(at 142.24 130.48 0)
 			(hide yes)
