File: hardware/lv_relay_drive.kicad_sch (KiCad schematic)
At the start: 15 parts, among them Q3 NMOS, Q5 NMOS, Q6 NMOS

Commit message: add holding voltage to lv_relay_drive block
Parts:
- added C14, C15, C16: C, symbol Device:C
- added R25, R26, R27: R_US, symbol Device:R_US
Connections:
- net DRV_AIR_NEG_OUT: now also C16.1, R27.2; no longer D10.1 (K), Q6.1 (D)
- net DRV_AIR_POS_OUT: now also C15.1, R26.2; no longer D8.1 (K), Q5.1 (D)
- net DRV_AIR_PRE_OUT: now also C14.1, R25.2; no longer D6.1 (K), Q3.1 (D)
- new net: C14.2, D6.1 (K), Q3.1 (D), R25.1
- new net: C15.2, D8.1 (K), Q5.1 (D), R26.1
- new net: C16.2, D10.1 (K), Q6.1 (D), R27.1
Other:
- note added: "Holding voltage"

Commit message: start power supply and logic sizing
Connections:
- net DRV_AIR_NEG_OUT: now also D10.1 (K)
- net DRV_AIR_POS_OUT: now also D8.1 (K)
- net DRV_AIR_PRE_OUT: now also D6.1 (K)
- net at C14.2, Q3.1 (D), R25.1: no longer D6.1 (K)
- net at C15.2, Q5.1 (D), R26.1: no longer D8.1 (K)
- net at C16.2, Q6.1 (D), R27.1: no longer D10.1 (K)
Other:
- moved on the sheet: C14, C15, C16, R25, R26, R27
